Commit message: Modify to remove warning when parsing URDF

File: intera_tools_description/urdf/connector_plate/connector_plate.xacro (robot description, xacro)
@@ -24,7 +24,7 @@
           <cylinder length="${rethink_connector_plate_length*2.0}" radius="0.04"/>
         </geometry>
-        <material name="darkred">
+        <!-- <material name="darkred">
           <color rgba=".5 .1 .1 1"/>
-        </material>
+        </material> -->
     </collision>
   </link>

File: intera_tools_description/urdf/electric_gripper/rethink_electric_gripper.xacro (robot description, xacro)
@@ -25,7 +25,7 @@
           <cylinder length="0.1" radius="0.029"/>
         </geometry>
-        <material name="darkred">
+	<!-- <material name="darkred">
           <color rgba=".5 .1 .1 1"/>
-        </material>
+        </material> -->
       </collision>
       <inertial>
@@ -119,5 +119,5 @@
       </joint>
       <actuator name="gripper_${gripper_side}1_motor1">
-        <hardwareInterface>hardware_interface/EffortJointInterface</hardwareInterface>
+        <!-- <hardwareInterface>hardware_interface/EffortJointInterface</hardwareInterface> -->
         <mechanicalReduction>1</mechanicalReduction>
       </actuator>
@@ -129,5 +129,5 @@
       </joint>
       <actuator name="gripper_${gripper_side}1_motor2">
-        <hardwareInterface>hardware_interface/EffortJointInterface</hardwareInterface>
+        <!-- <hardwareInterface>hardware_interface/EffortJointInterface</hardwareInterface> -->
         <mechanicalReduction>1</mechanicalReduction>
       </actuator>
